Commit message: Added LIDAR sensor, teleop keyboard integration, updated Dockerfile and README

File: colcon_ws/install/amr_description/share/amr_description/urdf/amr.urdf (robot description, URDF)
Before this commit: robot amr_bot, 3 links, 2 joints
Links:
- added link lidar_link; visual cylinder length=0.05 radius=0.05
Joints:
- removed joint base_to_wheel_left
- removed joint base_to_wheel_right
- added joint base_to_lidar: type fixed, parent base_link, child lidar_link, origin xyz=0 0 0.125 rpy=0 0 0
- added joint left_joint: type continuous, parent base_link, child wheel_left, origin xyz=-0.2 0.2 0 rpy=0 0 0, axis 0 1 0
- added joint right_joint: type continuous, parent base_link, child wheel_right, origin xyz=-0.2 -0.2 0 rpy=0 0 0, axis 0 1 0
